Commit message: Mujoco cobot launch

File: dual_arm_control/worlds/dual_panda_with_object.xml.xacro (robot description, xacro)
@@ -1,11 +1,29 @@
 <?xml version="1.0"?>
-<mujoco xmlns:xacro="http://www.ros.org/wiki/xacro" model="Dual Panda Scene with Object">
+<mujoco xmlns:xacro="http://ros.org/wiki/xacro" model="Dual Panda Scene with Object">
     <option timestep="0.001" gravity="0 0 -9.81" cone="elliptic" />
     <size njmax="500" nconmax="100" />
     <compiler angle="radian" />
+    <xacro:arg name="arm_id_0" default="L_panda" />
+    <xacro:arg name="x0" default="-0.5" />
+    <xacro:arg name="y0" default="0" />
+    <xacro:arg name="z0" default="0" />
+    <xacro:arg name="roll0" default="0" />
+    <xacro:arg name="pitch0" default="0" />
+    <xacro:arg name="yaw0" default="1.57" />
+    <xacro:arg name="arm_id_1" default="R_panda" />
+    <xacro:arg name="x1" default="0.5" />
+    <xacro:arg name="y1" default="0" />
+    <xacro:arg name="z1" default="0" />
+    <xacro:arg name="roll1" default="0" />
+    <xacro:arg name="pitch1" default="0" />
+    <xacro:arg name="yaw1" default="1.57" />
+    <xacro:arg name="use_suction_0" default="false" />
+    <xacro:arg name="use_suction_1" default="false" />
     <xacro:arg name="object_x" default="0.0" />
     <xacro:arg name="object_y" default="0.4" />
     <xacro:arg name="object_z" default="0.04" />
+    <xacro:property name="panda_shared_definitions_loaded" value="false" />
     <xacro:include filename="$(find franka_mujoco)/assets/xacro/panda.mujoco.xacro" />
+    <xacro:include filename="$(find franka_mujoco)/assets/xacro/panda_suction.mujoco.xacro" />
     <xacro:include filename="$(find dual_arm_control)/worlds/object.xacro" />
     <visual>
@@ -21,9 +39,29 @@
     </worldbody>
     <worldbody>
-        <xacro:panda_robot name="L_panda" pos="-0.5 0 0" rot="0 0 1.57" />
-        <xacro:panda_robot name="R_panda" pos="0.5 0 0" rot="0 0 1.57" />
+        <xacro:if value="$(arg use_suction_0)">
+            <xacro:panda_robot_suction name="$(arg arm_id_0)" pos="$(arg x0) $(arg y0) $(arg z0)" rot="$(arg roll0) $(arg pitch0) $(arg yaw0)" />
+        </xacro:if>
+        <xacro:unless value="$(arg use_suction_0)">
+            <xacro:panda_robot name="$(arg arm_id_0)" pos="$(arg x0) $(arg y0) $(arg z0)" rot="$(arg roll0) $(arg pitch0) $(arg yaw0)" />
+        </xacro:unless>
+        <xacro:if value="$(arg use_suction_1)">
+            <xacro:panda_robot_suction name="$(arg arm_id_1)" pos="$(arg x1) $(arg y1) $(arg z1)" rot="$(arg roll1) $(arg pitch1) $(arg yaw1)" />
+        </xacro:if>
+        <xacro:unless value="$(arg use_suction_1)">
+            <xacro:panda_robot name="$(arg arm_id_1)" pos="$(arg x1) $(arg y1) $(arg z1)" rot="$(arg roll1) $(arg pitch1) $(arg yaw1)" />
+        </xacro:unless>
         <xacro:graspable_box name="object_to_grasp" x="$(arg object_x)" y="$(arg object_y)" z="$(arg object_z)" />
     </worldbody>
-    <xacro:panda_extra name="L_panda" />
-    <xacro:panda_extra name="R_panda" />
+    <xacro:if value="$(arg use_suction_0)">
+        <xacro:panda_extra_suction name="$(arg arm_id_0)" />
+    </xacro:if>
+    <xacro:unless value="$(arg use_suction_0)">
+        <xacro:panda_extra name="$(arg arm_id_0)" />
+    </xacro:unless>
+    <xacro:if value="$(arg use_suction_1)">
+        <xacro:panda_extra_suction name="$(arg arm_id_1)" />
+    </xacro:if>
+    <xacro:unless value="$(arg use_suction_1)">
+        <xacro:panda_extra name="$(arg arm_id_1)" />
+    </xacro:unless>
 </mujoco>

Commit message: checker board update

File: dual_arm_control/worlds/dual_panda_with_object.xml.xacro (robot description, xacro)
@@ -30,6 +30,9 @@
     </visual>
     <asset>
-        <texture builtin="checker" height="512" name="texplane" rgb1=".2 .3 .4" rgb2=".1 .15 .2" type="2d" width="512" />
-        <material name="MatPlane" reflectance="0.05" shininess="0.01" specular="0.01" texrepeat="1 1" texture="texplane" texuniform="true" />
+        <!-- Modified texture for black and white chessboard pattern -->
+        <!-- rgb1 is Black (0 0 0), rgb2 is White (1 1 1) -->
+        <!-- texrepeat="50 50" creates 50x50 repeats over the 5m plane, making 10cm squares -->
+        <texture builtin="checker" height="512" name="texplane" rgb1="0 0 0" rgb2="1 1 1" type="2d" width="512" />
+        <material name="MatPlane" reflectance="0.05" shininess="0.01" specular="0.01" texrepeat="50 50" texture="texplane" texuniform="true" />
     </asset>
     <worldbody>

Commit message: update

File: dual_arm_control/worlds/dual_panda_with_object.xml.xacro (robot description, xacro)
@@ -34,5 +34,5 @@
         <!-- texrepeat="50 50" creates 50x50 repeats over the 5m plane, making 10cm squares -->
         <texture builtin="checker" height="512" name="texplane" rgb1="0 0 0" rgb2="1 1 1" type="2d" width="512" />
-        <material name="MatPlane" reflectance="0.05" shininess="0.01" specular="0.01" texrepeat="50 50" texture="texplane" texuniform="true" />
+        <material name="MatPlane" reflectance="0.05" shininess="0.01" specular="0.01" texrepeat="1 1" texture="texplane" texuniform="true" />
     </asset>
     <worldbody>
